Commit message: feat: add LiDAR sensor integration and update sensor visualization
- Added GPU LiDAR sensor with configurable parameters
- Updated IMU and LiDAR visual representations
- Set IMU color to blue and LiDAR color to purple for better visibility
- Adjusted sensor positions for optimal placement
- Added visual elements to SDF model for better visualization

File: src/world_01/models/diff_bot_sensors/model.urdf.xacro (robot description, xacro)
@@ -27,5 +27,5 @@
             </geometry>
             <material name="">
-                <color rgba="0.8 0.2 0.2 1"/>
+                <color rgba="0.8 0.2 0.2 0.8"/>
             </material>
         </visual>
@@ -48,5 +48,5 @@
             </geometry>
             <material name="">
-                <color rgba="0.2 0.2 0.2 1"/>
+                <color rgba="0.2 0.2 0.2 0.8"/>
             </material>
         </visual>
@@ -128,5 +128,5 @@
             </geometry>
             <material name="">
-                <color rgba="0.0 1.0 0.0 1.0"/>
+                <color rgba="0.0 0.0 1.0 1.0"/>  <!-- Blue -->
             </material>
         </visual>
@@ -141,3 +141,28 @@
         <child link="imu_link"/>
     </joint>
+    <!-- Lidar Link -->
+    <link name="lidar_link">
+        <inertial>
+            <mass value="0.001"/>
+            <inertia ixx="0.000001" ixy="0" ixz="0" iyy="0.000001" iyz="0" izz="0.000001"/>
+        </inertial>
+        <visual>
+            <geometry>
+                <box size="0.02 0.02 0.01"/>
+            </geometry>
+            <material name="">
+                <color rgba="0.5 0.0 0.5 1.0"/>  <!-- Purple -->
+            </material>
+        </visual>
+        <collision>
+            <geometry>
+                <box size="0.02 0.02 0.01"/>
+            </geometry>
+        </collision>
+    </link>
+    <joint name="lidar_joint" type="fixed">
+        <parent link="base_link"/>
+        <child link="lidar_link"/>
+        <origin xyz="0 0 0.15" rpy="0 0 0"/>
+    </joint>
 </robot>

Commit message: Updated root frame to odom instead of dummy link

File: src/world_01/models/diff_bot_sensors/model.urdf.xacro (robot description, xacro)
@@ -10,10 +10,10 @@
     <xacro:property name="caster_radius" value="0.05"/>
     <!-- Dummy link -->
-    <link name="dummy_link"></link>
+    <!-- <link name="dummy_link"></link>
     <joint name="dummy_joint" type="fixed">
         <parent link="dummy_link"/>
         <child link="base_link"/>
         <origin xyz="0 0 0" rpy="0 0 0"/>
-    </joint>
+    </joint> -->
     <!-- Base Link -->
     <link name="base_link">
